File: tuxkeychain.kicad_pcb (KiCad board)
At the start: 2 copper layers, 23.4 x 28.1 mm, 10 parts

Commit message: Remove old PCB stuff, change PCB to 4-layers, and improve README.
Parts:
- removed ? (x9): , Graphics
- removed ?: , DrillHole
Other:
- board outline removed
- copper layers 2 -> 4

Commit message: Enhance PDF generation by including silkscreen layers; add image generation workflow for KiCad
Other:
- board outline added: 34.6 x 25.5 mm
- board text added: "tmp"
Changed lines of the file:
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@@
 	)
 	(net 0 "")
+	(gr_rect
+		(start 84.2 45.1)
+		(end 118.8 70.6)
+		(stroke
+			(width 0.05)
+			(type default)
+		)
+		(fill no)
+		(layer "Edge.Cuts")
+	)
+	(gr_text "tmp\n"
+		(at 93.2 53.2 0)
+		(layer "F.SilkS")
+		(effects
+			(font
+				(size 1 1)
+				(thickness 0.1)
+			)
+			(justify left bottom)
+		)
+	)
 	(embedded_fonts no)
 )
