File: tuxkeychain.kicad_pcb (KiCad board)
At the start: 4 copper layers, 34.6 x 25.5 mm, 0 parts

Commit message: Added initial design files and artwork.
- Add attribution for Tux
- Setup PCB
- Add tux/ folder with files for the PCB art
Other:
- board outline removed
- copper layers 4 -> 6
- board text removed: "tmp"
Changed lines of the file:
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@@
 	)
 	(paper "A4")
+	(title_block
+		(title "Tux Keychain")
+		(date "2025-05-20")
+		(rev "1")
+		(company "All Things Linux 501(c)(3)")
+	)
 	(layers
 		(0 "F.Cu" signal)
 		(4 "In1.Cu" signal)
 		(6 "In2.Cu" signal)
+		(8 "In3.Cu" signal)
+		(10 "In4.Cu" signal)
 		(2 "B.Cu" signal)
 		(9 "F.Adhes" user "F.Adhesive")
@@
 			(layer "dielectric 2"
 				(type "core")
-				(thickness 1.24)
+				(thickness 0.535)
 				(material "FR4")
 				(epsilon_r 4.5)
@@
 			)
 			(layer "dielectric 3"
+				(type "prepreg")
+				(thickness 0.1)
+				(material "FR4")
+				(epsilon_r 4.5)
+				(loss_tangent 0.02)
+			)
+			(layer "In3.Cu"
+				(type "copper")
+				(thickness 0.035)
+			)
+			(layer "dielectric 4"
+				(type "core")
+				(thickness 0.535)
+				(material "FR4")
+				(epsilon_r 4.5)
+				(loss_tangent 0.02)
+			)
+			(layer "In4.Cu"
+				(type "copper")
+				(thickness 0.035)
+			)
+			(layer "dielectric 5"
 				(type "prepreg")
 				(thickness 0.1)
@@
 				(type "Bottom Silk Screen")
 			)
-			(copper_finish "None")
+			(copper_finish "ENIG")
 			(dielectric_constraints no)
 		)
@@
 	)
 	(net 0 "")
-	(gr_rect
-		(start 84.2 45.1)
-		(end 118.8 70.6)
-		(stroke
-			(width 0.05)
-			(type default)
-		)
-		(fill no)
-		(layer "Edge.Cuts")
-	)
-	(gr_text "tmp\n"
-		(at 93.2 53.2 0)
-		(layer "F.SilkS")
-		(effects
-			(font
-				(size 1 1)
-				(thickness 0.1)
-			)
-			(justify left bottom)
-		)
-	)
 	(embedded_fonts no)
 )

Commit message: Add PCB design and assign footprints
Parts:
- added C1: 2u2, Capacitor_SMD:C_0603_1608Metric, F.Cu at (96.9, 92.3)
- added C10: 22u, Capacitor_SMD:C_0603_1608Metric, F.Cu at (92.5, 87.8)
- added C11: 22u, Capacitor_SMD:C_0603_1608Metric, F.Cu at (92.5, 81.2)
- added C12: 100n, Capacitor_SMD:C_0603_1608Metric, F.Cu at (69.8, 103.8)
- added C13: 100n, Capacitor_SMD:C_0603_1608Metric, F.Cu at (80.5, 100.8)
- added C14: 100n, Capacitor_SMD:C_0603_1608Metric, F.Cu at (70.2, 88.7)
- added C15: 1u, Capacitor_SMD:C_0603_1608Metric, F.Cu at (79.2, 102.0)
- added C16: 1u, Capacitor_SMD:C_0603_1608Metric, F.Cu at (81.8, 99.5)
- added C17: 30p, Capacitor_SMD:C_0603_1608Metric, F.Cu at (77.5, 87.8)
- added C18: 30p, Capacitor_SMD:C_0603_1608Metric, F.Cu at (83.5, 88.2)
- added C2: 2u2, Capacitor_SMD:C_0603_1608Metric, F.Cu at (97.0, 86.5)
- added C3: 2u2, Capacitor_SMD:C_0603_1608Metric, F.Cu at (66.7, 99.6)
- added C4: 100n, Capacitor_SMD:C_0603_1608Metric, F.Cu at (69.8, 102.2)
- added C5: 100n, Capacitor_SMD:C_0603_1608Metric, F.Cu at (82.0, 92.5)
- added C6: 100n, Capacitor_SMD:C_0603_1608Metric, F.Cu at (72.5, 86.5)
- added C7: 100n, Capacitor_SMD:C_0603_1608Metric, F.Cu at (69.0, 90.0)
- added C8: 100n, Capacitor_SMD:C_0603_1608Metric, F.Cu at (67.8, 91.2)
- added C9: 22u, Capacitor_SMD:C_0603_1608Metric, F.Cu at (92.7, 93.6)
- added D1: LED (RED), LED_SMD:LED_0603_1608Metric, F.Cu at (58.0, 99.0)
- added F1: SMD0805B050TF, Fuse:Fuse_0805_2012Metric, F.Cu at (96.8, 98.2)
- added J1: Amphenol_10104110, Connector_USB:USB_Micro-B_Amphenol_10104110_Horizontal, F.Cu at (57.8, 86.2)
- added JP1: jumper, Jumper:SolderJumper-2_P1.3mm_Bridged_RoundedPad1.0x1.5mm, F.Cu at (57.9, 93.0)
- added L1: 2u2, Inductor_SMD:L_0805_2012Metric, F.Cu at (89.7, 95.3)
- added L2: 2u2, Inductor_SMD:L_0805_2012Metric, F.Cu at (89.5, 89.5)
- added L3: 2u2, Inductor_SMD:L_0805_2012Metric, F.Cu at (89.5, 82.9)
- added Q2: 2N7002, Package_TO_SOT_SMD:SOT-23, F.Cu at (61.8, 102.2)
- added R1: 11k, Resistor_SMD:R_0603_1608Metric, F.Cu at (92.7, 97.1)
- added R10: 120, Resistor_SMD:R_0603_1608Metric, F.Cu at (58.0, 100.8)
- added R11: 49k9, Resistor_SMD:R_0603_1608Metric, F.Cu at (61.0, 99.0)
- added R12: 49k9, Resistor_SMD:R_0603_1608Metric, F.Cu at (65.2, 98.2)
- added R2: 11k, Resistor_SMD:R_0603_1608Metric, F.Cu at (92.6, 91.2)
- added R3: 10k, Resistor_SMD:R_0603_1608Metric, F.Cu at (92.5, 84.8)
- added R4: 49k9, Resistor_SMD:R_0603_1608Metric, F.Cu at (92.7, 95.3)
- added R5: 36k, Resistor_SMD:R_0603_1608Metric, F.Cu at (92.6, 89.5)
- added R6: 8k2, Resistor_SMD:R_0603_1608Metric, F.Cu at (92.5, 83.0)
- added R7: 2k2, Resistor_SMD:R_0603_1608Metric, F.Cu at (77.8, 103.0)
- added R8: 2k2, Resistor_SMD:R_0603_1608Metric, F.Cu at (82.2, 103.8)
- added R9: 3k3, Resistor_SMD:R_0603_1608Metric, F.Cu at (94.0, 101.5)
- added SW1: B3U-1000P, Button_Switch_SMD:SW_SPST_B3U-1000P, F.Cu at (58.0, 96.2)
- added U1: JW5211, Package_TO_SOT_SMD:SOT-23-5, F.Cu at (96.4, 95.3)
- added U2: JW5211, Package_TO_SOT_SMD:SOT-23-5, F.Cu at (96.5, 89.5)
- added U3: JW5211, Package_TO_SOT_SMD:SOT-23-5, F.Cu at (96.5, 83.0)
- added U4: F1C100s, tuxkeychain:QFN-88_EP_10x10_Pitch0.4mm, F.Cu at (74.0, 96.0)
- added U5: AT25SF081B-SSHD-T, Package_SO:SOIC-8_3.9x4.9mm_P1.27mm, F.Cu at (88.8, 101.0)
- added Y1: 24MHz, Crystal:Crystal_SMD_3225-4Pin_3.2x2.5mm, F.Cu at (80.0, 90.0)
Routing:
- net +3V3: track 0.00 -> 90.0 mm, vias 0 -> 8
- net +1V1: track 0.00 -> 58.1 mm, vias 0 -> 4
- net +2V6: track 0.00 -> 52.8 mm, vias 0 -> 3
- net VBUS: track 0.00 -> 42.1 mm, vias 0 -> 2
- net GND: track 0.00 -> 36.7 mm, vias 0 -> 7
- net SPI_CS: track 0.00 -> 26.2 mm, vias 0 -> 2
- net +5V: track 0.00 -> 22.4 mm
- net SPI_MISO: track 0.00 -> 21.7 mm, vias 0 -> 2
- net ~{RESET}: track 0.00 -> 20.3 mm, vias 0 -> 2
- net SPI_MOSI: track 0.00 -> 15.9 mm, vias 0 -> 2
- net D-: track 0.00 -> 15.7 mm
- net D+: track 0.00 -> 15.3 mm
- net SPI_CLK: track 0.00 -> 14.9 mm, vias 0 -> 2
- net STATUS: track 0.00 -> 13.0 mm, vias 0 -> 2
- net Net-(J1-Shield): track 0.00 -> 10.9 mm
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- added copper zone on B.Cu, net GND
- added copper zone on F.Cu, net GND
- added copper zone on In1.Cu, net GND
- added copper zone on In2.Cu, net GND
- added copper zone on In3.Cu, net GND
- added copper zone on In4.Cu, net GND
Other:
- board outline added: 45 x 25 mm
- board text added: "Tux Keychain Prototype Rev. ${REVISION}"

Commit message: Change USB footprint to a more available model
Parts:
- J1: value Amphenol_10104110 -> Amphenol_10104111; footprint Connector_USB:USB_Micro-B_Amphenol_10104110_Horizontal -> tuxkeychain:CONN_10104111-0001LF_AMP
- moved J1 0.83 mm to (57.0, 86.2)
Changed lines of the file:
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@@
 		)
 	)
-	(footprint "Connector_USB:USB_Micro-B_Amphenol_10104110_Horizontal"
+	(footprint "tuxkeychain:CONN_10104111-0001LF_AMP"
 		(layer "F.Cu")
-		(at 57.8 86.15 -90)
-		(descr "USB Micro-B, horizontal, https://cdn.amphenol-icc.com/media/wysiwyg/files/drawing/10104110.pdf")
-		(tags "USB Micro B horizontal")
+		(at 56.9701 86.15 -90)
+		(tags "10104111-0001LF ")
 		(property "Reference" "J1"
-			(at 0 -3.55 90)
+			(at 0 -2.7202 270)
+			(unlocked yes)
 			(layer "F.SilkS")
 			(hide yes)
@@
 			)
 		)
-		(property "Value" "Amphenol_10104110"
-			(at 0 5.35 90)
+		(property "Value" "Amphenol_10104111"
+			(at 0 -2.7202 270)
+			(unlocked yes)
 			(layer "F.Fab")
 			(effects
@@
 		(property "Datasheet" ""
 			(at 0 0 270)
-			(unlocked yes)
 			(layer "F.Fab")
 			(hide yes)
@@
 			)
 		)
-		(property "Description" "USB Micro Type B connector"
+		(property "Description" ""
 			(at 0 0 270)
-			(unlocked yes)
 			(layer "F.Fab")
 			(hide yes)
@@
 		(attr smd)
 		(fp_line
-			(start -3.86 4.16)
-			(end 3.86 4.16)
-			(stroke
-				(width 0.12)
-				(type solid)
-			)
-			(layer "F.SilkS")
-		)
-		(fp_line
-			(start -3.86 4.16)
-			(end -3.86 2.55)
-			(stroke
-				(width 0.12)
-				(type solid)
-			)
-			(layer "F.SilkS")
-		)
-		(fp_line
-			(start 3.86 4.16)
-			(end 3.86 2.55)
-			(stroke
-				(width 0.12)
-				(type solid)
-			)
-			(layer "F.SilkS")
-		)
-		(fp_line
-			(start -3.86 0.05)
-			(end -3.86 -1.66)
-			(stroke
-				(width 0.12)
-				(type solid)
-			)
-			(layer "F.SilkS")
-		)
-		(fp_line
-			(start 3.86 0.05)
-			(end 3.86 -1.66)
-			(stroke
-				(width 0.12)
-				(type solid)
-			)
-			(layer "F.SilkS")
-		)
-		(fp_line
-			(start -3.86 -1.66)
-			(end -1.8 -1.66)
-			(stroke
-				(width 0.12)
-				(type solid)
-			)
-			(layer "F.SilkS")
-		)
-		(fp_line
-			(start -1.8 -1.66)
-			(end -1.8 -2.25)
-			(stroke
-				(width 0.12)
-				(type solid)
-			)
-			(layer "F.SilkS")
-		)
-		(fp_line
-			(start 3.86 -1.66)
-			(end 1.8 -1.66)
-			(stroke
-				(width 0.12)
-				(type solid)
-			)
-			(layer "F.SilkS")
-		)
-		(fp_line
-			(start -5.4 4.549999)
-			(end 5.4 4.549999)
-			(stroke
-				(width 0.05)
+			(start -4.5212 2.9972)
+			(end 4.5212 2.9972)
+			(stroke
+				(width 0.1524)
+				(type solid)
+			)
+			(layer "F.SilkS")
+		)
+		(fp_line
+			(start 4.5212 2.9972)
+			(end 4.5212 1.415039)
+			(stroke
+				(width 0.1524)
+				(type solid)
+			)
+			(layer "F.SilkS")
+		)
+		(fp_line
+			(start -4.5212 1.415039)
+			(end -4.5212 2.9972)
+			(stroke
+				(width 0.1524)
+				(type solid)
+			)
+			(layer "F.SilkS")
+		)
+		(fp_line
+			(start 4.5212 -1.155441)
+			(end 4.5212 -2.9972)
+			(stroke
+				(width 0.1524)
+				(type solid)
+			)
+			(layer "F.SilkS")
+		)
+		(fp_line
+			(start -4.5212 -2.9972)
+			(end -4.5212 -1.155441)
+			(stroke
+				(width 0.1524)
+				(type solid)
+			)
+			(layer "F.SilkS")
+		)
+		(fp_line
+			(start -1.83594 -2.9972)
+			(end -4.5212 -2.9972)
+			(stroke
+				(width 0.1524)
+				(type solid)
+			)
+			(layer "F.SilkS")
+		)
+		(fp_line
+			(start 4.5212 -2.9972)
+			(end 1.83594 -2.9972)
+			(stroke
+				(width 0.1524)
+				(type solid)
+			)
+			(layer "F.SilkS")
+		)
+		(fp_circle
+			(center -4.5212 -2.9972)
+			(end -4.1402 -2.9972)
+			(stroke
+				(width 0.508)
+				(type solid)
+			)
+			(fill no)
+			(layer "F.SilkS")
+		)
+		(fp_line
+			(start -5.1597 3.1242)
+			(end 5.1597 3.1242)
+			(stroke
+				(width 0.1524)
 				(type solid)
 			)
@@
 		)
 		(fp_line
-			(start 5.4 4.549999)
-			(end 5.4 -2.75)
-			(stroke
-				(width 0.05)
+			(start 5.1597 3.1242)
+			(end 5.1597 -3.6727)
+			(stroke
+				(width 0.1524)
 				(type solid)
 			)
@@
 		)
 		(fp_line
-			(start -5.4 -2.75)
-			(end -5.4 4.549999)
-			(stroke
-				(width 0.05)
+			(start -5.1597 -3.6727)
+			(end -5.1597 3.1242)
+			(stroke
+				(width 0.1524)
 				(type solid)
 			)
@@
 		)
 		(fp_line
-			(start 5.4 -2.75)
-			(end -5.4 -2.75)
-			(stroke
-				(width 0.05)
+			(start 5.1597 -3.6727)
+			(end -5.1597 -3.6727)
+			(stroke
+				(width 0.1524)
 				(type solid)
 			)
@@
 		)
 		(fp_line
-			(start -3.75 4.05)
-			(end -3.75 -1.55)
-			(stroke
-				(width 0.1)
-				(type solid)
-			)
-			(layer "F.Fab")
-		)
-		(fp_line
-			(start 3.75 4.05)
-			(end -3.75 4.05)
-			(stroke
-				(width 0.1)
-				(type solid)
-			)
-			(layer "F.Fab")
-		)
-		(fp_line
-			(start -2.6 2.75)
-			(end 2.6 2.75)
-			(stroke
-				(width 0.1)
-				(type solid)
-			)
-			(layer "F.Fab")
-		)
-		(fp_line
-			(start -3.75 -1.55)
-			(end 3.75 -1.55)
-			(stroke
-				(width 0.1)
-				(type solid)
-			)
-			(layer "F.Fab")
-		)
-		(fp_line
-			(start 3.75 -1.55)
-			(end 3.75 4.05)
-			(stroke
-				(width 0.1)
-				(type solid)
-			)
-			(layer "F.Fab")
-		)
-		(fp_line
-			(start -1.3 -1.85)
-			(end -0.9 -2.25)
-			(stroke
-				(width 0.1)
-				(type solid)
-			)
-			(layer "F.Fab")
-		)
-		(fp_line
-			(start -1.7 -2.25)
-			(end -1.3 -1.85)
-			(stroke
-				(width 0.1)
-				(type solid)
-			)
-			(layer "F.Fab")
-		)
-		(fp_line
-			(start -0.9 -2.25)
-			(end -1.7 -2.25)
-			(stroke
-				(width 0.1)
-				(type solid)
-			)
-			(layer "F.Fab")
-		)
-		(fp_text user "PCB edge"
-			(at 0 2.75 90)
-			(layer "Dwgs.User")
-			(effects
-				(font
-					(size 0.5 0.5)
-					(thickness 0.08)
-				)
-			)
+			(start -4.3942 2.8702)
+			(end 4.3942 2.8702)
+			(stroke
+				(width 0.0254)
+				(type solid)
+			)
+			(layer "F.Fab")
+		)
+		(fp_line
+			(start 4.3942 2.8702)
+			(end 4.3942 -2.8702)
+			(stroke
+				(width 0.0254)
+				(type solid)
+			)
+			(layer "F.Fab")
+		)
+		(fp_line
+			(start -4.3942 -2.8702)
+			(end -4.3942 2.8702)
+			(stroke
+				(width 0.0254)
+				(type solid)
+			)
+			(layer "F.Fab")
+		)
+		(fp_line
+			(start 4.3942 -2.8702)
+			(end -4.3942 -2.8702)
+			(stroke
+				(width 0.0254)
+				(type solid)
+			)
+			(layer "F.Fab")
+		)
+		(fp_circle
+			(center -1.3 -4.6252)
+			(end -0.919 -4.6252)
+			(stroke
+				(width 0.508)
+				(type solid)
+			)
+			(fill no)
+			(layer "F.Fab")
 		)
 		(fp_text user "${REFERENCE}"
-			(at 0 -0.199999 90)
+			(at 0 -2.7202 270)
+			(unlocked yes)
 			(layer "F.Fab")
 			(effects
@@
 		)
 		(pad "1" smd rect
-			(at -1.3 -1.55 270)
-			(size 0.4 1.4)
+			(at -1.3 -2.7202 270)
+			(size 0.4064 1.397)
 			(layers "F.Cu" "F.Mask" "F.Paste")
 			(net 9 "VBUS")
@@
 		)
 		(pad "2" smd rect
-			(at -0.65 -1.55 270)
-			(size 0.4 1.4)
+			(at -0.649999 -2.7202 270)
+			(size 0.4064 1.397)
 			(layers "F.Cu" "F.Mask" "F.Paste")
 			(net 10 "D-")
@@
 		)
 		(pad "3" smd rect
-			(at 0 -1.550001 270)
-			(size 0.4 1.4)
+			(at 0 -2.7202 270)
+			(size 0.4064 1.397)
 			(layers "F.Cu" "F.Mask" "F.Paste")
 			(net 13 "D+")
@@
 		)
 		(pad "4" smd rect
-			(at 0.65 -1.55 270)
-			(size 0.4 1.4)
+			(at 0.649999 -2.7202 270)
+			(size 0.4064 1.397)
 			(layers "F.Cu" "F.Mask" "F.Paste")
 			(net 12 "unconnected-(J1-ID-Pad4)")
@@
 		)
 		(pad "5" smd rect
-			(at 1.3 -1.55 270)
-			(size 0.4 1.4)
+			(at 1.3 -2.7202 270)
+			(size 0.4064 1.397)
 			(layers "F.Cu" "F.Mask" "F.Paste")
 			(net 2 "GND")
@@
 		)
 		(pad "6" smd rect
-			(at -3.75 1.3 270)
-			(size 2.3 1.9)
+			(at -3.75 0.129799 270)
+			(size 2.3114 1.905)
 			(layers "F.Cu" "F.Mask" "F.Paste")
 			(net 11 "Net-(J1-Shield)")
@@
 		)
 		(pad "6" smd rect
-			(at -1.15 1.3 270)
-			(size 1.8 1.9)
+			(at -1.15 0.129799 270)
+			(size 1.8034 1.905)
 			(layers "F.Cu" "F.Mask" "F.Paste")
 			(net 11 "Net-(J1-Shield)")
@@
 		)
 		(pad "6" smd rect
-			(at 1.15 1.3 270)
-			(size 1.8 1.9)
+			(at 1.15 0.129799 270)
+			(size 1.8034 1.905)
 			(layers "F.Cu" "F.Mask" "F.Paste")
 			(net 11 "Net-(J1-Shield)")
@@
 		)
 		(pad "6" smd rect
-			(at 3.75 1.3 270)
-			(size 2.3 1.9)
+			(at 3.75 0.129799 270)
+			(size 2.3114 1.905)
 			(layers "F.Cu" "F.Mask" "F.Paste")
 			(net 11 "Net-(J1-Shield)")
@@
 		)
 		(embedded_fonts no)
-		(model "${KICAD9_3DMODEL_DIR}/Connector_USB.3dshapes/USB_Micro-B_Molex_47346-0001.step"
+		(model "${KIPRJMOD}/lib/10104111C.stp"
 			(offset
-				(xyz 0 0 0)
+				(xyz 0 1 1.5)
 			)
 			(scale
@@
 			)
 			(rotate
-				(xyz 0 0 0)
-			)
-		)
+				(xyz -90 -0 -0)
+			)
+		)
