File: tuxkeychain.kicad_pcb (KiCad board)
At the start: 6 copper layers, 45 x 25 mm, 45 parts, among them J1 Amphenol_10104111, Q2 2N7002, SW1 B3U-1000P, U1 JW5211, U2 JW5211, U3 JW5211, U4 F1C100s, U5 AT25SF081B-SSHD-T, Y1 24MHz

Commit message: Change flash chip
Parts:
- removed U5: AT25SF081B-SSHD-T, Package_SO:SOIC-8_3.9x4.9mm_P1.27mm
- added U6: W25Q128JVS, Package_SO:SOIC-8_5.3x5.3mm_P1.27mm, F.Cu at (89.0, 101.0)
- moved R9 2.03 mm to (96.0, 101.8)
Routing:
- net +3V3: track 90.0 -> 93.5 mm
- net SPI_MOSI: track 15.9 -> 14.7 mm
- net SPI_CLK: track 14.9 -> 13.8 mm
- net SPI_MISO: track 21.7 -> 22.5 mm
