File: tuxkeychain.kicad_sch (KiCad schematic)
At the start: 45 parts, among them J1 USB_B_Micro, Q1 Q_PMOS_GSD, SW1 SW_Push, U1 F1C100s, U2 JW5211, U3 JW5211, U4 JW5211, U5 AT25SF081-SSHD-X, Y1 24MHz

Commit message: Reannotate symbols
Parts:
- renumbered C4 to C10, C5 to C11, C11 to C13, C10 to C14, C9 to C15, C8 to C16, C6 to C17, C7 to C18, C13 to C3, C14 to C4, C15 to C5, C16 to C6, C17 to C7, C18 to C8, C3 to C9, R9 to R10, R10 to R11, R11 to R12, R12 to R9, U2 to U1, U3 to U2, U4 to U3, U1 to U4

Commit message: Refactor TuxKeychain Schematic: Update PMOS to NMOS, Adjust Power Symbols
- Changed PMOS transistor symbols and properties to NMOS in tuxkeychain.kicad_sch.
- Updated power symbols from +2V5 to +3V3 and +5V to GND, reflecting correct voltage levels.
- Modified descriptions and keywords for clarity and accuracy.
- Added new global label "STATUS" for better schematic organization.
- Cleaned up unused symbols and properties to streamline the schematic.
Parts:
- Q1: value Q_PMOS_GSD -> Q_NMOS_GSD; symbol Transistor_FET:Q_PMOS_GSD -> Transistor_FET:Q_NMOS_GSD
Connections:
- net STATUS: now also Q1.1 (G), R11.1
- net +2V5 renamed +2V6
Other:
- note removed: "actually 2.6v TODO: cry"
Changed lines of the file:
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@@
 		)
 	)
-	(text "actually 2.6v\nTODO: cry"
-		(exclude_from_sim no)
-		(at 86.995 55.245 0)
-		(effects
-			(font
-				(size 1.27 1.27)
-			)
-		)
-	)
 	(junction
 		(at 77.47 38.1)
@@
 		)
 	)
+	(global_label "STATUS"
+		(shape bidirectional)
+		(at 193.04 146.05 270)
+		(effects
+			(font
+				(size 1.27 1.27)
+			)
+			(justify right)
+		)
+		(property "Intersheetrefs" "${INTERSHEET_REFS}"
+			(at 193.04 146.05 90)
+			(effects
+				(font
+					(size 1.27 1.27)
+				)
+				(hide yes)
+			)
+		)
+	)
 	(global_label "SPI_MOSI"
 		(shape bidirectional)
@@
 	)
 	(symbol
-		(lib_id "Transistor_FET:Q_PMOS_GSD")
+		(lib_id "Transistor_FET:Q_NMOS_GSD")
 		(at 179.07 146.05 0)
 		(mirror y)
@@
 			)
 		)
-		(property "Value" "Q_PMOS_GSD"
+		(property "Value" "Q_NMOS_GSD"
 			(at 172.72 147.3199 0)
 			(effects
@@
 			)
 		)
-		(property "Description" "P-MOSFET transistor, gate/source/drain"
+		(property "Description" "N-MOSFET transistor, gate/source/drain"
 			(at 179.07 146.05 0)
 			(effects
@@
 	)
 	(symbol
-		(lib_id "power:+2V5")
+		(lib_id "tuxkeychain:+2V6")
 		(at 50.8 125.73 0)
 		(mirror y)
@@
 		(on_board yes)
 		(dnp no)
-		(property "Reference" "#PWR08"
+		(property "Reference" "#PWR8"
 			(at 50.8 129.54 0)
 			(effects
@@
 			)
 		)
-		(property "Value" "+2V5"
+		(property "Value" "+2V6"
 			(at 46.99 124.46 0)
 			(effects
@@
 			)
 		)
-		(property "Description" "Power symbol creates a global label with name \"+2V5\""
+		(property "Description" "Power symbol creates a global label with name \"+2V6\""
 			(at 50.8 125.73 0)
 			(effects
@@
 			(project "tuxkeychain"
 				(path "/b08030bf-1ef2-4626-81f6-c1cc66f6d9b4"
-					(reference "#PWR08")
+					(reference "#PWR8")
 					(unit 1)
 				)
@@
 	)
 	(symbol
-		(lib_id "power:+2V5")
+		(lib_id "tuxkeychain:+2V6")
 		(at 92.71 118.11 0)
 		(unit 1)
@@
 		(on_board yes)
 		(dnp no)
-		(property "Reference" "#PWR020"
+		(property "Reference" "#PWR20"
 			(at 92.71 121.92 0)
 			(effects
@@
 			)
 		)
-		(property "Value" "+2V5"
+		(property "Value" "+2V6"
 			(at 96.52 116.84 0)
 			(effects
@@
 			)
 		)
-		(property "Description" "Power symbol creates a global label with name \"+2V5\""
+		(property "Description" "Power symbol creates a global label with name \"+2V6\""
 			(at 92.71 118.11 0)
 			(effects
@@
 			(project "tuxkeychain"
 				(path "/b08030bf-1ef2-4626-81f6-c1cc66f6d9b4"
-					(reference "#PWR020")
+					(reference "#PWR20")
 					(unit 1)
 				)
@@
 	)
 	(symbol
-		(lib_id "power:+2V5")
+		(lib_id "tuxkeychain:+2V6")
 		(at 77.47 57.15 0)
 		(unit 1)
@@
 		(dnp no)
 		(fields_autoplaced yes)
-		(property "Reference" "#PWR017"
+		(property "Reference" "#PWR17"
 			(at 77.47 60.96 0)
 			(effects
@@
 			)
 		)
-		(property "Value" "+2V5"
+		(property "Value" "+2V6"
 			(at 77.47 52.07 0)
 			(effects
@@
 			)
 		)
-		(property "Description" "Power symbol creates a global label with name \"+2V5\""
+		(property "Description" "Power symbol creates a global label with name \"+2V6\""
 			(at 77.47 57.15 0)
 			(effects
@@
 			(project ""
 				(path "/b08030bf-1ef2-4626-81f6-c1cc66f6d9b4"
-					(reference "#PWR017")
+					(reference "#PWR17")
 					(unit 1)
 				)

Commit message: Update component values in TuxKeychain schematic
Parts:
- J1: value USB_B_Micro -> Amphenol_10104110
- U5: value AT25SF081-SSHD-X -> AT25SF081B-SSHD-T
Changed lines of the file:
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@@
 			)
 		)
-		(property "Value" "AT25SF081-SSHD-X"
+		(property "Value" "AT25SF081B-SSHD-T"
 			(at 154.94 179.0699 0)
 			(effects
@@
 			)
 		)
-		(property "Value" "USB_B_Micro"
+		(property "Value" "Amphenol_10104110"
 			(at 33.02 157.48 0)
 			(effects

Commit message: Add PCB design and assign footprints
Parts:
- removed Q1: Q_NMOS_GSD, symbol Transistor_FET:Q_NMOS_GSD
- added Q2: 2N7002, Package_TO_SOT_SMD:SOT-23, symbol Transistor_FET:2N7002
- C1, C10, C11, C12, C13, C14, C15, C16, C17, C18, C2, C3, C4, C5, C6, C7, C8, C9: footprint (none) -> Capacitor_SMD:C_0603_1608Metric
- D1: footprint (none) -> LED_SMD:LED_0603_1608Metric
- F1: value Polyfuse -> SMD0805B050TF; footprint (none) -> Fuse:Fuse_0805_2012Metric
- L1, L2, L3: footprint (none) -> Inductor_SMD:L_0805_2012Metric
- R1, R10, R11, R12, R2, R3, R4, R5, R6, R7, R8, R9: footprint (none) -> Resistor_SMD:R_0603_1608Metric
- SW1: value SW_Push -> B3U-1000P; footprint (none) -> Button_Switch_SMD:SW_SPST_B3U-1000P
- Y1: footprint (none) -> Crystal:Crystal_SMD_3225-4Pin_3.2x2.5mm
Connections:
- net GND: now also Q2.2 (S)
- net STATUS: now also Q2.1 (G)
- net at R10.1: now also Q2.3 (D)
Other:
- note added: "crystal that we use: CF4024M00012001"
Changed lines of the file:
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@@
 	(text "maybe we can save costs by removing this polyfuse,\nsure maybe itll fry someones devices but thats\ntheir fucking problem"
 		(exclude_from_sim no)
-		(at 93.345 17.145 0)
+		(at 92.71 16.51 0)
 		(effects
 			(font
@@
 		)
 	)
+	(text "crystal that we use: CF4024M00012001"
+		(exclude_from_sim no)
+		(at 264.795 13.97 0)
+		(effects
+			(font
+				(size 1.27 1.27)
+			)
+		)
+	)
 	(text "you *probably* dont need to open it\nbut its just for prototype failsafe"
 		(exclude_from_sim no)
@@
 	(text "TODO: move this the fuck out of here\nthis doesnt belong in a fucking\ncorner theres a reason global labels exist"
 		(exclude_from_sim no)
-		(at 242.57 16.51 0)
+		(at 227.965 20.955 0)
 		(effects
 			(font
@@
 			)
 		)
-		(property "Footprint" ""
+		(property "Footprint" "Capacitor_SMD:C_0603_1608Metric"
 			(at 274.32 32.7152 0)
 			(effects
@@
 	)
 	(symbol
-		(lib_id "Transistor_FET:Q_NMOS_GSD")
-		(at 179.07 146.05 0)
-		(mirror y)
-		(unit 1)
-		(exclude_from_sim no)
-		(in_bom yes)
-		(on_board yes)
-		(dnp no)
-		(fields_autoplaced yes)
-		(property "Reference" "Q1"
-			(at 172.72 144.7799 0)
-			(effects
-				(font
-					(size 1.27 1.27)
-				)
-				(justify left)
-			)
-		)
-		(property "Value" "Q_NMOS_GSD"
-			(at 172.72 147.3199 0)
-			(effects
-				(font
-					(size 1.27 1.27)
-				)
-				(justify left)
-			)
-		)
-		(property "Footprint" ""
-			(at 173.99 143.51 0)
-			(effects
-				(font
-					(size 1.27 1.27)
-				)
-				(hide yes)
-			)
-		)
-		(property "Datasheet" "~"
-			(at 179.07 146.05 0)
-			(effects
-				(font
-					(size 1.27 1.27)
-				)
-				(hide yes)
-			)
-		)
-		(property "Description" "N-MOSFET transistor, gate/source/drain"
-			(at 179.07 146.05 0)
-			(effects
-				(font
-					(size 1.27 1.27)
-				)
-				(hide yes)
-			)
-		)
-		(pin "1"
-		)
-		(pin "2"
-		)
-		(pin "3"
-		)
-		(instances
-			(project ""
-				(path "/b08030bf-1ef2-4626-81f6-c1cc66f6d9b4"
-					(reference "Q1")
-					(unit 1)
-				)
-			)
-		)
-	)
-	(symbol
 		(lib_id "power:GND")
 		(at 101.6 123.19 0)
@@
 			)
 		)
-		(property "Footprint" ""
+		(property "Footprint" "Capacitor_SMD:C_0603_1608Metric"
 			(at 78.4352 69.85 0)
 			(effects
@@
 			)
 		)
-		(property "Footprint" ""
+		(property "Footprint" "Capacitor_SMD:C_0603_1608Metric"
 			(at 274.32 23.1648 0)
 			(effects
@@
 			)
 		)
-		(property "Footprint" ""
+		(property "Footprint" "Resistor_SMD:R_0603_1608Metric"
 			(at 99.822 138.43 90)
 			(effects
@@
 			)
 		)
-		(property "Footprint" ""
+		(property "Footprint" "Inductor_SMD:L_0805_2012Metric"
 			(at 73.66 59.69 0)
 			(effects
@@
 	)
 	(symbol
+		(lib_id "Transistor_FET:2N7002")
+		(at 179.07 146.05 0)
+		(mirror y)
+		(unit 1)
+		(exclude_from_sim no)
+		(in_bom yes)
+		(on_board yes)
+		(dnp no)
+		(fields_autoplaced yes)
+		(property "Reference" "Q2"
+			(at 172.72 144.7799 0)
+			(effects
+				(font
+					(size 1.27 1.27)
+				)
+				(justify left)
+			)
+		)
+		(property "Value" "2N7002"
+			(at 172.72 147.3199 0)
+			(effects
+				(font
+					(size 1.27 1.27)
+				)
+				(justify left)
+			)
+		)
+		(property "Footprint" "Package_TO_SOT_SMD:SOT-23"
+			(at 173.99 147.955 0)
+			(effects
+				(font
+					(size 1.27 1.27)
+					(italic yes)
+				)
+				(justify left)
+				(hide yes)
+			)
+		)
+		(property "Datasheet" "https://www.onsemi.com/pub/Collateral/NDS7002A-D.PDF"
+			(at 173.99 149.86 0)
+			(effects
+				(font
+					(size 1.27 1.27)
+				)
+				(justify left)
+				(hide yes)
+			)
+		)
+		(property "Description" "0.115A Id, 60V Vds, N-Channel MOSFET, SOT-23"
+			(at 179.07 146.05 0)
+			(effects
+				(font
+					(size 1.27 1.27)
+				)
+				(hide yes)
+			)
+		)
+		(pin "1"
+		)
+		(pin "2"
+		)
+		(pin "3"
+		)
+		(instances
+			(project ""
+				(path "/b08030bf-1ef2-4626-81f6-c1cc66f6d9b4"
+					(reference "Q2")
+					(unit 1)
+				)
+			)
+		)
+	)
+	(symbol
 		(lib_id "power:VBUS")
 		(at 40.64 162.56 270)
@@
 			)
 		)
-		(property "Footprint" ""
+		(property "Footprint" "Capacitor_SMD:C_0603_1608Metric"
 			(at 96.52 114.3 0)
 			(effects
@@
 			)
 		)
-		(property "Footprint" ""
+		(property "Footprint" "Resistor_SMD:R_0603_1608Metric"
 			(at 70.358 41.91 90)
 			(effects
@@
 			)
 		)
-		(property "Footprint" ""
+		(property "Footprint" "Capacitor_SMD:C_0603_1608Metric"
 			(at 96.52 111.76 0)
 			(effects
@@
 			)
 		)
-		(property "Value" "SW_Push"
+		(property "Value" "B3U-1000P"
 			(at 227.33 152.3999 90)
 			(effects
@@
 			)
 		)
-		(property "Footprint" ""
+		(property "Footprint" "Button_Switch_SMD:SW_SPST_B3U-1000P"
 			(at 228.6 151.13 0)
 			(effects
@@
 			)
 		)
-		(property "Footprint" ""
+		(property "Footprint" "Resistor_SMD:R_0603_1608Metric"
 			(at 225.298 142.24 90)
 			(effects
@@
 			)
 		)
-		(property "Value" "Polyfuse"
+		(property "Value" "SMD0805B050TF"
 			(at 60.96 17.78 90)
 			(effects
@@
 			)
 		)
-		(property "Footprint" ""
+		(property "Footprint" "Fuse:Fuse_0805_2012Metric"
 			(at 66.04 20.32 0)
 			(effects
@@
 			)
 		)
-		(property "Footprint" ""
+		(property "Footprint" "Capacitor_SMD:C_0603_1608Metric"
 			(at 48.26 111.76 0)
 			(effects
@@
 			)
 		)
-		(property "Footprint" ""
+		(property "Footprint" "Resistor_SMD:R_0603_1608Metric"
 			(at 70.358 87.63 90)
 			(effects
@@
 			)
 		)
-		(property "Footprint" ""
+		(property "Footprint" "Capacitor_SMD:C_0603_1608Metric"
 			(at 40.3352 45.72 0)
 			(effects
@@
 			)
 		)
-		(property "Footprint" ""
+		(property "Footprint" "Capacitor_SMD:C_0603_1608Metric"
 			(at 48.26 116.84 0)
 			(effects
@@
 			)
 		)
-		(property "Footprint" ""
+		(property "Footprint" "Capacitor_SMD:C_0603_1608Metric"
 			(at 48.26 109.22 0)
 			(effects
@@
 			)
 		)
-		(property "Footprint" ""
+		(property "Footprint" "Resistor_SMD:R_0603_1608Metric"
 			(at 132.842 166.37 90)
 			(effects
@@
 			)
 		)
-		(property "Footprint" ""
+		(property "Footprint" "Inductor_SMD:L_0805_2012Metric"
 			(at 73.66 35.56 0)
 			(effects
@@
 			)
 		)
-		(property "Footprint" ""
+		(property "Footprint" "Resistor_SMD:R_0603_1608Metric"
 			(at 203.708 142.24 90)
 			(effects
@@
 			)
 		)
-		(property "Footprint" ""
+		(property "Footprint" "LED_SMD:LED_0603_1608Metric"
 			(at 195.58 138.43 0)
 			(effects
@@
 			)
 		)
-		(property "Footprint" ""
+		(property "Footprint" "Resistor_SMD:R_0603_1608Metric"
 			(at 97.79 131.318 90)
 			(effects
@@
 			)
 		)
-		(property "Footprint" ""
+		(property "Footprint" "Capacitor_SMD:C_0603_1608Metric"
 			(at 48.26 127 0)
 			(effects
@@
 			)
 		)
-		(property "Footprint" ""
+		(property "Footprint" "Capacitor_SMD:C_0603_1608Metric"
 			(at 96.52 109.22 0)
 			(effects
@@
 			)
 		)
-		(property "Footprint" ""
+		(property "Footprint" "Capacitor_SMD:C_0603_1608Metric"
 			(at 48.26 119.38 0)
 			(effects
@@
 			)
 		)
-		(property "Footprint" ""
+		(property "Footprint" "Resistor_SMD:R_0603_1608Metric"
 			(at 73.66 36.322 90)
 			(effects
@@
 			)
 		)
-		(property "Footprint" ""
+		(property "Footprint" "Resistor_SMD:R_0603_1608Metric"
 			(at 73.66 82.042 90)
 			(effects
@@
 			)
 		)
-		(property "Footprint" ""
+		(property "Footprint" "Inductor_SMD:L_0805_2012Metric"
 			(at 73.66 81.28 0)
 			(effects
@@
 			)
 		)
-		(property "Footprint" ""
+		(property "Footprint" "Capacitor_SMD:C_0603_1608Metric"
 			(at 78.4352 45.72 0)
 			(effects
@@
 			)
 		)
-		(property "Footprint" ""
+		(property "Footprint" "Resistor_SMD:R_0603_1608Metric"
 			(at 70.358 66.04 90)
 			(effects
@@
 			)
 		)
-		(property "Footprint" ""
+		(property "Footprint" "Resistor_SMD:R_0603_1608Metric"
 			(at 73.66 60.452 90)
 			(effects
@@
 			)
 		)
-		(property "Footprint" ""
+		(property "Footprint" "Resistor_SMD:R_0603_1608Metric"
 			(at 184.15 140.208 90)
 			(effects
@@
 			)
 		)
-		(property "Footprint" ""
+		(property "Footprint" "Capacitor_SMD:C_0603_1608Metric"
 			(at 48.26 114.3 0)
 			(effects
@@
 			)
 		)
-		(property "Footprint" ""
+		(property "Footprint" "Capacitor_SMD:C_0603_1608Metric"
 			(at 96.52 127 0)
 			(effects
@@
 			)
 		)
-		(property "Footprint" ""
+		(property "Footprint" "Capacitor_SMD:C_0603_1608Metric"
 			(at 33.3248 45.72 0)
 			(effects
@@
 			)
 		)
-		(property "Footprint" ""
+		(property "Footprint" "Capacitor_SMD:C_0603_1608Metric"
 			(at 78.4352 91.44 0)
 			(effects
@@
 			)
 		)
-		(property "Footprint" ""
+		(property "Footprint" "Crystal:Crystal_SMD_3225-4Pin_3.2x2.5mm"
 			(at 264.16 27.94 0)
 			(effects
@@
 			)
 		)
-		(property "Footprint" ""
+		(property "Footprint" "Capacitor_SMD:C_0603_1608Metric"
 			(at 96.52 119.38 0)
 			(effects

Commit message: Change USB footprint to a more available model
Parts:
- J1: value Amphenol_10104110 -> Amphenol_10104111; footprint Connector_USB:USB_Micro-B_Amphenol_10104110_Horizontal -> tuxkeychain:CONN_10104111-0001LF_AMP
Changed lines of the file:
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@@
 			)
 		)
-		(property "Value" "Amphenol_10104110"
+		(property "Value" "Amphenol_10104111"
 			(at 33.02 157.48 0)
 			(effects
@@
 			)
 		)
-		(property "Footprint" "Connector_USB:USB_Micro-B_Amphenol_10104110_Horizontal"
+		(property "Footprint" "tuxkeychain:CONN_10104111-0001LF_AMP"
 			(at 36.83 168.91 0)
 			(effects

Commit message: Add TODO for unsoldered SMT header to enhance hacking potential
Other:
- note added: "TODO: add a unsoldered SMT header for hacking potential"
Changed lines of the file:
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@@
+		)
+	)
+	(text "TODO: add a unsoldered SMT header for hacking potential"
+		(exclude_from_sim no)
+		(at 247.015 164.465 0)
+		(effects
+			(font
+				(size 1.27 1.27)
+			)
 		)
 	)

Commit message: Change flash chip
Parts:
- removed U5: AT25SF081B-SSHD-T, Package_SO:SOIC-8_3.9x4.9mm_P1.27mm, symbol Memory_Flash:AT25SF081-SSHD-X
- added U6: W25Q128JVS, Package_SO:SOIC-8_5.3x5.3mm_P1.27mm, symbol Memory_Flash:W25Q128JVS
Connections:
- net +3V3: now also U6.3 (~{WP}/IO_{2}), U6.7 (~{HOLD}/~{RESET}/IO_{3}), U6.8 (VCC)
- net GND: now also U6.4 (GND)
- net SPI_CLK: now also U6.6 (CLK)
- net SPI_CS: now also U6.1 (~{CS})
- net SPI_MISO: now also U6.2 (DO/IO_{1})
- net SPI_MOSI: now also U6.5 (DI/IO_{0})
Other:
- note removed: "sshd reference"
Changed lines of the file:
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@@
 		)
 	)
-	(text "sshd reference\n"
-		(exclude_from_sim no)
-		(at 161.29 182.245 0)
-		(effects
-			(font
-				(size 1.27 1.27)
-			)
-		)
-	)
 	(text "maybe they are\ncursed, or maybe\nthe designer was\nlazy.\nTODO: exorcism\n"
 		(exclude_from_sim no)
@@
 	)
 	(junction
+		(at 135.89 182.88)
+		(diameter 0)
+		(color 0 0 0 0)
+	)
+	(junction
 		(at 77.47 78.74)
 		(diameter 0)
@@
 	)
 	(junction
-		(at 135.89 182.88)
-		(diameter 0)
-		(color 0 0 0 0)
-	)
-	(junction
 		(at 77.47 62.23)
 		(diameter 0)
@@
 	)
 	(symbol
-		(lib_id "Memory_Flash:AT25SF081-SSHD-X")
-		(at 146.05 177.8 0)
-		(unit 1)
-		(exclude_from_sim no)
-		(in_bom yes)
-		(on_board yes)
-		(dnp no)
-		(fields_autoplaced yes)
-		(property "Reference" "U5"
-			(at 154.94 176.5299 0)
-			(effects
-				(font
-					(size 1.27 1.27)
-				)
-				(justify left)
-			)
-		)
-		(property "Value" "AT25SF081B-SSHD-T"
-			(at 154.94 179.0699 0)
-			(effects
-				(font
-					(size 1.27 1.27)
-				)
-				(justify left)
-			)
-		)
-		(property "Footprint" "Package_SO:SOIC-8_3.9x4.9mm_P1.27mm"
-			(at 146.05 193.04 0)
-			(effects
-				(font
-					(size 1.27 1.27)
-				)
-				(hide yes)
-			)
-		)
-		(property "Datasheet" "https://www.adestotech.com/wp-content/uploads/DS-AT25SF081_045.pdf"
-			(at 146.05 177.8 0)
-			(effects
-				(font
-					(size 1.27 1.27)
-				)
-				(hide yes)
-			)
-		)
-		(property "Description" "8-Mbit, 2.5V Minimum SPI Serial Flash Memory with Dual-I/O and Quad-I/O Support, SOIC-8"
-			(at 146.05 177.8 0)
-			(effects
-				(font
-					(size 1.27 1.27)
-				)
-				(hide yes)
-			)
-		)
-		(pin "1"
-		)
-		(pin "2"
-		)
-		(pin "7"
-		)
-		(pin "3"
-		)
-		(pin "5"
-		)
-		(pin "6"
-		)
-		(pin "4"
-		)
-		(pin "8"
-		)
-		(instances
-			(project ""
-				(path "/b08030bf-1ef2-4626-81f6-c1cc66f6d9b4"
-					(reference "U5")
-					(unit 1)
-				)
-			)
-		)
-	)
-	(symbol
 		(lib_id "power:GND")
 		(at 69.85 142.24 0)
@@
 					(unit 1)
 				)
+			)
+		)
+	)
+	(symbol
+		(lib_id "Memory_Flash:W25Q128JVS")
+		(at 146.05 177.8 0)
+		(unit 1)
+		(exclude_from_sim no)
+		(in_bom yes)
+		(on_board yes)
+		(dnp no)
+		(fields_autoplaced yes)
+		(property "Reference" "U6"
+			(at 157.48 176.5299 0)
+			(effects
+				(font
+					(size 1.27 1.27)
+				)
+				(justify left)
+			)
+		)
+		(property "Value" "W25Q128JVS"
+			(at 157.48 179.0699 0)
+			(effects
+				(font
+					(size 1.27 1.27)
+				)
+				(justify left)
+			)
+		)
+		(property "Footprint" "Package_SO:SOIC-8_5.3x5.3mm_P1.27mm"
+			(at 146.05 154.94 0)
+			(effects
+				(font
+					(size 1.27 1.27)
+				)
+				(hide yes)
+			)
+		)
+		(property "Datasheet" "https://www.winbond.com/resource-files/w25q128jv_dtr%20revc%2003272018%20plus.pdf"
+			(at 146.05 152.4 0)
+			(effects
+				(font
+					(size 1.27 1.27)
+				)
+				(hide yes)
+			)
+		)
+		(property "Description" "128Mbit / 16MiB Serial Flash Memory, Standard/Dual/Quad SPI, 2.7-3.6V, SOIC-8"
+			(at 146.05 149.86 0)
+			(effects
+				(font
+					(size 1.27 1.27)
+				)
+				(hide yes)
+			)
+		)
+		(pin "4"
+		)
+		(pin "6"
+		)
+		(pin "3"
+		)
+		(pin "5"
+		)
+		(pin "7"
+		)
+		(pin "2"
+		)
+		(pin "8"
+		)
+		(pin "1"
+		)
+		(instances
+			(project ""
+				(path "/b08030bf-1ef2-4626-81f6-c1cc66f6d9b4"
+					(reference "U6")
+					(unit 1)
+				)

Commit message: Refactor schematic comments
Other:
- note added: "in the spirit of blinkenlights, this will not be removed"
- note removed: "TODO: remove this..? TODO: decide if i should remove this"
- note removed: "we probably don't need jtag"
Changed lines of the file:
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@@
 		)
 	)
-	(text "TODO: remove this..?\nTODO: decide if i should remove this"
+	(text "in the spirit of blinkenlights,\nthis will not be removed"
 		(exclude_from_sim no)
 		(at 157.48 137.795 0)
@@
 	(text "TODO: add a unsoldered SMT header for hacking potential"
 		(exclude_from_sim no)
-		(at 247.015 164.465 0)
+		(at 253.365 163.83 0)
 		(effects
 			(font
@@
 		(effects
 			(font
-				(size 1.27 1.27)
-			)
-		)
-	)
-	(text "we probably\ndon't need jtag"
-		(exclude_from_sim no)
-		(at 271.78 75.565 0)
-		(effects
-			(font
